Commit message: kinematics Chain update

File: capstone_ws/src/turret_description/urdf/ADT.urdf (robot description, URDF)
Before this commit: robot adt, 6 links, 5 joints
Links:
- removed link Camera_Link
- removed link Camera_Pitch_Link
- removed link Pitch_Link
- removed link Rail_Link
- removed link Yaw_Link
- removed link base_link
- added link Base_link, mass 1.19126257965004; collision mesh filename=package://ADT/meshes/Base_link.STL; visual mesh filename=package://ADT/meshes/Base_link.STL
- added link Camera_link, mass 0.0463212382951515; collision mesh filename=package://ADT/meshes/Camera_link.STL; visual mesh filename=package://ADT/meshes/Camera_link.STL
- added link Camera_pitch_link, mass 0.0488857805315246; collision mesh filename=package://ADT/meshes/Camera_pitch_link.STL; visual mesh filename=package://ADT/meshes/Camera_pitch_link.STL
- added link Pitch_link, mass 0.110851272025115; collision mesh filename=package://ADT/meshes/Pitch_link.STL; visual mesh filename=package://ADT/meshes/Pitch_link.STL
- added link Rail_link, mass 0.0461878510377165; collision mesh filename=package://ADT/meshes/Rail_link.STL; visual mesh filename=package://ADT/meshes/Rail_link.STL
- added link Yaw_link, mass 0.792271578967464; collision mesh filename=package://ADT/meshes/Yaw_link.STL; visual mesh filename=package://ADT/meshes/Yaw_link.STL
Joints:
- removed joint Camera_Link_joint
- removed joint Camera_Pitch_Link_joint
- removed joint Pitch_Link_joint
- removed joint Rail_Link_joint
- removed joint Yaw_Link_joint
- added joint Camera_link_joint: type fixed, parent Camera_pitch_link, child Camera_link, origin xyz=0.041 -0.0043929 0.0010012 rpy=0 -2.6267E-05 0, axis 0 0 0
- added joint Camera_pitch_link_joint: type revolute, parent Yaw_link, child Camera_pitch_link, origin xyz=0.001 0 0.4091 rpy=0 0 0, axis 0 -1 0, limit lower=0 upper=0 effort=0 velocity=0
- added joint Pitch_link_joint: type revolute, parent Yaw_link, child Pitch_link, origin xyz=-0.00030345 0 0.156 rpy=0 0 0, axis 0 1 0, limit lower=0 upper=0 effort=0 velocity=0
- added joint Rail_link_joint: type fixed, parent Pitch_link, child Rail_link, origin xyz=0 0 -0.0395 rpy=0 0 0, axis 0 0 0
- added joint Yaw_link_joint: type revolute, parent Base_link, child Yaw_link, origin xyz=0.00087547 -0.010086 0.2234 rpy=0 0 0.017045, axis 0 0 -1, limit lower=0 upper=0 effort=0 velocity=0
